File: InertialUnits/alim33.sch (KiCad schematic (older format))
At the start: 5 parts, among them U13 AP1117

Commit message: Modification axis on Inertial sensors
Parts:
- removed U13: AP1117, symbol AP1117
- added U1: TLV1117, symbol TLV1117
Changed lines of the file:
@@
-EESchema Schematic File Version 2  date lun. 31 mars 2014 21:58:22 CEST
+EESchema Schematic File Version 2
 LIBS:power
 LIBS:device
@@
 LIBS:perso
 LIBS:inertialSensors-cache
-EELAYER 25  0
+EELAYER 24 0
 EELAYER END
-$Descr A4 11700 8267
+$Descr A4 11693 8268
 encoding utf-8
 Sheet 3 4
@@
 F 0 "C27" H 3000 2725 50  0000 L CNN
 F 1 "22uF" H 3000 2525 50  0000 L CNN
+F 2 "" H 2950 2650 60  0001 C CNN
+F 3 "" H 2950 2650 60  0001 C CNN
 	1    2950 2650
 	1    0    0    -1
@@
 F 0 "C10" H 1950 2650 50  0000 L CNN
 F 1 "10u" H 1950 2450 50  0000 L CNN
+F 2 "" H 1900 2550 60  0001 C CNN
+F 3 "" H 1900 2550 60  0001 C CNN
 	1    1900 2550
 	1    0    0    -1
 $EndComp
 $Comp
-L GND #PWR5
+L GND #PWR7
 U 1 1 5301DF7C
 P 4850 2950
-F 0 "#PWR5" H 4850 2950 30  0001 C CNN
+F 0 "#PWR7" H 4850 2950 30  0001 C CNN
 F 1 "GND" H 4850 2880 30  0001 C CNN
+F 2 "" H 4850 2950 60  0001 C CNN
+F 3 "" H 4850 2950 60  0001 C CNN
 	1    4850 2950
 	0    -1   -1   0
@@
 F 0 "D2" H 4500 3050 50  0000 C CNN
 F 1 "LED" H 4500 2850 50  0000 C CNN
+F 2 "" H 4500 2950 60  0001 C CNN
+F 3 "" H 4500 2950 60  0001 C CNN
 	1    4500 2950
 	1    0    0    -1
@@
 F 0 "R45" V 4080 2950 50  0000 C CNN
 F 1 "150" V 4000 2950 50  0000 C CNN
+F 2 "" H 4000 2950 60  0001 C CNN
+F 3 "" H 4000 2950 60  0001 C CNN
 	1    4000 2950
 	0    -1   -1   0
 $EndComp
 $Comp
-L GND #PWR4
+L GND #PWR6
 U 1 1 5301D3F5
 P 2950 3000
-F 0 "#PWR4" H 2950 3000 30  0001 C CNN
+F 0 "#PWR6" H 2950 3000 30  0001 C CNN
 F 1 "GND" H 2950 2930 30  0001 C CNN
+F 2 "" H 2950 3000 60  0001 C CNN
+F 3 "" H 2950 3000 60  0001 C CNN
 	1    2950 3000
-	1    0    0    -1
-$EndComp
-$Comp
-L AP1117 U13
-U 1 1 5301D3C4
-P 2450 2250
-F 0 "U13" H 2000 1750 60  0000 C CNN
-F 1 "AP1117" H 3100 1700 60  0000 C CNN
-	1    2450 2250
 	1    0    0    -1
 $EndComp
@@
 5V
 $Comp
-L GND #PWR2
+L GND #PWR4
 U 1 1 52FB371E
 P 1900 3050
-F 0 "#PWR2" H 1900 3050 30  0001 C CNN
+F 0 "#PWR4" H 1900 3050 30  0001 C CNN
 F 1 "GND" H 1900 2980 30  0001 C CNN
+F 2 "" H 1900 3050 60  0001 C CNN
+F 3 "" H 1900 3050 60  0001 C CNN
 	1    1900 3050
 	1    0    0    -1
 $EndComp
 $Comp
-L GND #PWR3
+L GND #PWR5
 U 1 1 52FB3715
 P 2450 3000
-F 0 "#PWR3" H 2450 3000 30  0001 C CNN
+F 0 "#PWR5" H 2450 3000 30  0001 C CNN
 F 1 "GND" H 2450 2930 30  0001 C CNN
+F 2 "" H 2450 3000 60  0001 C CNN
+F 3 "" H 2450 3000 60  0001 C CNN
 	1    2450 3000
 	1    0    0    -1
 $EndComp
+$Comp
+L TLV1117 U1
+U 1 1 5358F891
+P 2450 2300
+F 0 "U1" H 2000 1900 60  0000 C CNN
+F 1 "TLV1117" H 2850 2000 60  0000 C CNN
+F 2 "" H 2450 2300 60  0000 C CNN
+F 3 "" H 2450 2300 60  0000 C CNN
+	1    2450 2300
+	1    0    0    -1
+$EndComp
